File: Boards/MainBoard/CAN.kicad_sch (KiCad schematic)
At the start: 21 parts, among them IC5 MCP2515-e_ST, IC6 ISO1042BDWVR, Y1 8MHz

Commit message: Add Clearance To Main/CtrlBd, Increase main DCDC to 20w
Parts:
- PS2: footprint REC10K-AW -> InverterCom:REC10K-AW
Changed lines of the file:
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@@
 			)
 		)
-		(property "Footprint" "REC10K-AW"
+		(property "Footprint" "InverterCom:REC10K-AW"
 			(at 92.71 248.59 0)
 			(effects

Commit message: layout control boards, add baseplate, refine mechanical layout
Parts:
- PS2: footprint InverterCom:REC10K-AW -> REC10K-AW
Changed lines of the file:
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@@
 			)
 		)
-		(property "Footprint" "InverterCom:REC10K-AW"
+		(property "Footprint" "REC10K-AW"
 			(at 92.71 248.59 0)
 			(effects
