File: Boards/MainBoard/MainBoard.kicad_pcb (KiCad board)
At the start: 2 copper layers, 297.5 x 60 mm, 128 parts, among them IC1 MAX22530AWE+, IC13 DRDNB21D-7, IC14 DRDNB21D-7, IC2 MAX22530AWE+, IC5 MCP2515-e_ST, IC6 ISO1042BDWVR, J1 Conn_02x08_Counter_Clockwise, J11 Conn_02x10_Counter_Clockwise, J12 Conn_02x10_Counter_Clockwise, J13 Conn_02x10_Counter_Clockwise, J14 Conn_02x10_Counter_Clockwise, J2 Conn_02x08_Counter_Clockwise, J3 Conn_02x08_Counter_Clockwise, J4 TBP01R1-508-06BE, J5 Conn_02x10_Counter_Clockwise, J6 TBP01R1-508-06BE, K1 AWHSH105D00G, K2 AWHSH105D00G, K3 AWHSH105D00G, K4 AWHSH105D00G, Y1 8MHz

Commit message: layout control boards, add baseplate, refine mechanical layout
Parts:
- J6: value TBP01R1-508-06BE -> TBP01R2-508-06BE; footprint InverterCom:TBP01R150806BE -> InverterCom:TBP01R250806BE; moved to B.Cu
- moved H3 10.0 mm to (100.0, 45.0)
- moved H5 10.0 mm to (190.0, 45.0)
- moved J6 7.37 mm to (5.00, 39.0)
- moved H7 6.00 mm to (291.0, 48.0)
- moved H1 4.50 mm to (7.50, 48.0)
- moved H4 2.00 mm to (7.00, 5.00)
- moved J13 1.77 mm to (134.9, 45.0)
- moved K3 0.82 mm to (269.2, 46.0)
- moved K4 0.82 mm to (248.2, 44.0)
Other:
- outline, holes or cut-outs redrawn
- board text removed: "CHANGE THIS TO VERTICAL TERMINAL - PUT ON BACK OF PCB FACING DOWN."

Commit message: Layout mainboard, add EMI filter caps
Parts:
- removed K4: AWHSH105D00G, InverterCom:AWHSH105D00G
- added C148: UCM1H101MCL1GS, InverterCom:CAPAE660X800N, F.Cu at (185.0, 55.0)
- added C149: UCM1H101MCL1GS, InverterCom:CAPAE660X800N, F.Cu at (92.3, 55.0)
- added C150: UCM1H101MCL1GS, InverterCom:CAPAE660X800N, F.Cu at (114.8, 45.0)
- added C151: UCM1H101MCL1GS, InverterCom:CAPAE660X800N, F.Cu at (194.9, 55.0)
- added C152: UCM1H101MCL1GS, InverterCom:CAPAE660X800N, F.Cu at (102.2, 55.0)
- added C153: UCM1H101MCL1GS, InverterCom:CAPAE660X800N, F.Cu at (124.8, 45.0)
- added C154: UCM1H101MCL1GS, InverterCom:CAPAE660X800N, F.Cu at (204.8, 55.0)
- added C155: UCM1H101MCL1GS, InverterCom:CAPAE660X800N, F.Cu at (204.2, 45.0)
- added C156: UCM1H101MCL1GS, InverterCom:CAPAE660X800N, F.Cu at (115.0, 55.0)
- added C157: UCM1H101MCL1GS, InverterCom:CAPAE660X800N, F.Cu at (214.7, 55.0)
- added C158: UCM1H101MCL1GS, InverterCom:CAPAE660X800N, F.Cu at (214.2, 45.0)
- added C159: UCM1H101MCL1GS, InverterCom:CAPAE660X800N, F.Cu at (124.9, 55.0)
- added G***: LOGO, InverterCom:HIGHVOLTAGE_20mm, F.Cu at (170.5, 47.5)
- C25: moved to F.Cu
- moved C139 15.5 mm to (255.5, 42.5), turned to 0 degrees
- moved K3 12.0 mm to (281.0, 43.7), turned to 90 degrees
- moved K2 11.8 mm to (269.0, 11.2), turned to -90 degrees
- moved K1 10.4 mm to (250.0, 14.3), turned to -90 degrees
- moved C125 10.0 mm to (255.5, 47.0), turned to 0 degrees
- moved C29 5.76 mm to (146.4, 10.0), turned to 180 degrees
- moved TP1 4.03 mm to (40.0, 14.5)
- moved C25 1.95 mm to (146.4, 10.0), turned to 180 degrees
- moved C137 1.56 mm to (280.6, 49.0)
- moved IC13 1.06 mm to (267.2, 4.25), turned to 90 degrees
- moved PS1 1.00 mm to (74.2, 26.6)
- moved R8 1.00 mm to (148.0, 6.00)
- moved C3 0.50 mm to (68.5, 25.6)
- moved C4 0.50 mm to (68.5, 25.6)
- moved R98 0.50 mm to (16.4, 36.5)
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Connections:
- IC14 pad 1: Net-(IC14-C1/A1) -> unconnected-(IC14-C1/A1-Pad1)
- IC14 pad 6: /DRIVE_ENABLE_A -> /GND_A
- J1 pad 16: /+12V_SWITCHED_A -> /+12V_A
- J11 pad 4: /DRIVE_ENABLE_A -> unconnected-(J11-Pin_4-Pad4)
- J13 pad 7: unconnected-(J13-Pin_7-Pad7) -> /RESET
- J13 pad 8: unconnected-(J13-Pin_8-Pad8) -> /READY
- J13 pad 9: unconnected-(J13-Pin_9-Pad9) -> /FAULT
- J14 pad 5: /CAN_5V_OUT -> unconnected-(J14-Pin_5-Pad5)
- J2 pad 16: /+12V_SWITCHED_A -> /+12V_A
- J3 pad 16: /+12V_SWITCHED_A -> /+12V_A
- J5 pad 16: /+12V_A -> unconnected-(J5-Pin_16-Pad16)
- J5 pad 19: /+12V_SWITCHED_A -> unconnected-(J5-Pin_19-Pad19)
Routing:
- net /FAULT: track 0.00 -> 210.0 mm, vias 0 -> 3
- net /READY: track 0.00 -> 209.3 mm, vias 0 -> 5
- net /RESET: track 0.00 -> 203.1 mm, vias 0 -> 5
- net /PH_U_H: track 0.00 -> 113.8 mm, vias 0 -> 2
- net /PH_W_L: track 0.00 -> 113.7 mm, vias 0 -> 1
- net /PH_U_L: track 0.00 -> 113.1 mm, vias 0 -> 2
- net /PH_W_H: track 0.00 -> 109.2 mm, vias 0 -> 1
- net /RELAY_3_A: track 0.00 -> 69.9 mm, vias 0 -> 2
- net /RELAY1_COM: track 0.00 -> 68.6 mm
- net /RELAY3_COM: track 0.00 -> 58.5 mm
- net /OutputRelays/+5V_A_INT_2: track 0.00 -> 56.4 mm, vias 0 -> 2
- net /SPI1_SCK_A: track 0.00 -> 52.9 mm, vias 0 -> 4
- net /SPI1_TX_A: track 0.00 -> 48.4 mm, vias 0 -> 4
- net /SPI1_CAN_CS_A: track 0.00 -> 47.8 mm, vias 0 -> 4
- net /ADC_1/VoltageSenseInputStage3/LV_OUT: track 0.00 -> 46.7 mm, vias 0 -> 2
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- added copper zone on In2.Cu, net /+12V_A
- added copper zone on In3.Cu, net /+3.3V_A
- added copper zone on In2.Cu, net /+5V_Y
- added copper zone on In3.Cu, net /CAN_5V_OUT
- added copper zone on B.Cu, net /CAN_GND
- added copper zone on F.Cu, net /CAN_GND
- added copper zone on In1.Cu, net /CAN_GND
- added copper zone on In4.Cu, net /CAN_GND
- added copper zone on B.Cu, net /GND_A
- added copper zone on F.Cu, net /GND_A
- added copper zone on In1.Cu, net /GND_A
- added copper zone on In4.Cu, net /GND_A
- added copper zone on B.Cu, net /GND_U
- added copper zone on F.Cu, net /GND_U
- added copper zone on In1.Cu, net /GND_U
- added copper zone on In2.Cu, net /GND_U
- added copper zone on In3.Cu, net /GND_U
- added copper zone on In4.Cu, net /GND_U
- added copper zone on B.Cu, net /ISENSE_GND_Y
- added copper zone on F.Cu, net /ISENSE_GND_Y
- added copper zone on In1.Cu, net /ISENSE_GND_Y
- added copper zone on In4.Cu, net /ISENSE_GND_Y
Other:
- copper layers 2 -> 6
- board text added: "AUX OUTPUT RELAYS"
- board text added: "CONN. TO PH U GATE DRIVER"
- board text added: "CONN. TO PH V GATE DRIVER"
- board text added: "CONN. TO PH W GATE DRIVER"
- board text added: "DANGER HAZARDOUS VOLTAGES PRESENT REMOVE POWER BEFORE SERVICING"
- board text added: "DESIGNED BY THOMAS LIAO"
- board text added: "GND +5V DC U V W"
- board text added: "GND DC U V W GND"
- board text added: "ISOLATED CANBUS"
- board text added: "ISOLATED CURRENT SENSE"
- board text added: "ISOLATED VOLTAGE SENSE"
- board text added: "ISOLATION BARRIER DO NOT CROSS"
- board text added: "TRACTION INVERTER, GEN 5, MAIN INTERFACE BOARD, REVISION 1, 1200VMAX, 800V WORKING"

Commit message: fix connector pinout
Parts:
- moved J12 23.1 mm to (82.8, 40.0), turned to -90 degrees
- moved J13 23.0 mm to (157.8, 42.5), turned to -90 degrees
- moved J1 17.9 mm to (47.2, 54.8), turned to -90 degrees
- moved J2 17.9 mm to (137.2, 54.8), turned to -90 degrees
- moved J3 17.9 mm to (227.2, 54.8), turned to -90 degrees
Routing:
- net /PH_U_H: track 113.8 -> 93.5 mm
- net /PH_U_L: track 113.1 -> 96.2 mm
- net /RESET: track 203.1 -> 213.2 mm, vias 5 -> 4
- net /FAULT: track 210.0 -> 218.2 mm, vias 3 -> 5
- net /PH_W_H: track 109.2 -> 116.4 mm, vias 1 -> 2
- net /SPI1_CAN_INT_A: track 42.1 -> 47.6 mm
- net /READY: track 209.3 -> 214.5 mm
- net /PH_V_L: track 13.4 -> 8.63 mm
- net /SPI2_RX_A: track 35.3 -> 38.9 mm
- net /PH_V_H: track 13.0 -> 16.6 mm, vias 0 -> 2
- net /SPI2_ADC2_CS_A: track 24.9 -> 28.5 mm
- net /SPI1_CAN_CS_A: track 47.8 -> 44.3 mm
- net /SPI2_TX_A: track 36.9 -> 33.3 mm, vias 2 -> 3
- net /PH_W_L: track 113.7 -> 117.1 mm, vias 1 -> 2
- net /SPI2_SCK_A: track 36.2 -> 38.8 mm, vias 2 -> 3
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Other:
- board text added: "1->"
- board text added: "<-1"
