File: Boards/MainBoard/MainBoard.kicad_pcb (KiCad board)
At the start: 6 copper layers, 297.5 x 60 mm, 140 parts, among them IC1 MAX22530AWE+, IC13 DRDNB21D-7, IC14 DRDNB21D-7, IC2 MAX22530AWE+, IC5 MCP2515-e_ST, IC6 ISO1042BDWVR, J1 Conn_02x08_Counter_Clockwise, J11 Conn_02x10_Counter_Clockwise, J12 Conn_02x10_Counter_Clockwise, J13 Conn_02x10_Counter_Clockwise, J14 Conn_02x10_Counter_Clockwise, J2 Conn_02x08_Counter_Clockwise, J3 Conn_02x08_Counter_Clockwise, J4 TBP01R1-508-06BE, J5 Conn_02x10_Counter_Clockwise, J6 TBP01R2-508-06BE, K1 AWHSH105D00G, K2 AWHSH105D00G, K3 AWHSH105D00G, Y1 8MHz

Commit message: Add Clearance To Main/CtrlBd, Increase main DCDC to 20w
Parts:
- H1, H7: footprint MountingHole:MountingHole_5.3mm_M5 -> MountingHole:MountingHole_3.2mm_M3
- H3, H4, H5, H8: footprint MountingHole:MountingHole_5.3mm_M5 -> MountingHole:MountingHole_4.3mm_M4
- moved C137 41.0 mm to (242.0, 35.0)
- moved PS13 40.5 mm to (228.2, 38.1)
- moved C138 39.6 mm to (242.0, 41.0)
- moved H7 24.7 mm to (266.5, 51.0)
- moved H1 16.3 mm to (23.5, 51.0)
- moved K3 13.2 mm to (267.8, 43.7), turned to 0 degrees
- moved C125 9.71 mm to (250.0, 39.0)
- moved C139 9.71 mm to (250.0, 34.5)
- moved IC14 9.71 mm to (252.5, 43.0)
- moved R96 2.00 mm to (27.4, 35.0)
- moved R97 2.00 mm to (22.0, 35.0)
- moved R98 1.50 mm to (16.4, 35.0)
- moved K1 1.12 mm to (250.0, 13.2)
Routing:
- net /RELAY_3_A: track 69.9 -> 57.8 mm
- net Net-(IC14-C2/A2): track 27.1 -> 15.7 mm
- net /RELAY3_NO: track 21.9 -> 33.0 mm
- net /OutputRelays/+5V_A_INT: track 44.2 -> 39.1 mm
- net /GND_A: track 17.8 -> 20.2 mm, vias 42 -> 39
- net /OutputRelays/+5V_A_INT_2: track 56.4 -> 55.3 mm
- net /PH_W_VSENSE_U: track 11.2 -> 10.3 mm
- net Net-(R95-Pad2): track 2.45 -> 3.28 mm
- net /RELAY3_COM: track 58.5 -> 57.8 mm
Other:
- outline, holes or cut-outs redrawn
