File: Boards/MainBoard/MainBoard.kicad_sch (KiCad schematic)
At the start: 28 parts, among them J1 Conn_02x08_Counter_Clockwise, J11 Conn_02x10_Counter_Clockwise, J12 Conn_02x10_Counter_Clockwise, J13 Conn_02x10_Counter_Clockwise, J14 Conn_02x10_Counter_Clockwise, J2 Conn_02x08_Counter_Clockwise, J3 Conn_02x08_Counter_Clockwise, J4 TBP01R1-508-06BE, J5 Conn_02x10_Counter_Clockwise, J6 TBP01R2-508-06BE

Commit message: Add Clearance To Main/CtrlBd, Increase main DCDC to 20w
Parts:
- H1, H7: footprint MountingHole:MountingHole_5.3mm_M5 -> MountingHole:MountingHole_3.2mm_M3
- H3, H4, H5, H8: footprint MountingHole:MountingHole_5.3mm_M5 -> MountingHole:MountingHole_4.3mm_M4
- J6: footprint TBP01R250806BE -> InverterCom:TBP01R250806BE
Changed lines of the file:
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@@
 			)
 		)
-		(property "Footprint" "MountingHole:MountingHole_5.3mm_M5"
+		(property "Footprint" "MountingHole:MountingHole_4.3mm_M4"
 			(at 254 33.02 0)
 			(effects
@@
 			)
 		)
-		(property "Footprint" "MountingHole:MountingHole_5.3mm_M5"
+		(property "Footprint" "MountingHole:MountingHole_3.2mm_M3"
 			(at 254 25.4 0)
 			(effects
@@
 			)
 		)
-		(property "Footprint" "MountingHole:MountingHole_5.3mm_M5"
+		(property "Footprint" "MountingHole:MountingHole_4.3mm_M4"
 			(at 254 52.07 0)
 			(effects
@@
 			)
 		)
-		(property "Footprint" "MountingHole:MountingHole_5.3mm_M5"
+		(property "Footprint" "MountingHole:MountingHole_3.2mm_M3"
 			(at 254 60.96 0)
 			(effects
@@
 			)
 		)
-		(property "Footprint" "MountingHole:MountingHole_5.3mm_M5"
+		(property "Footprint" "MountingHole:MountingHole_4.3mm_M4"
 			(at 254 45.72 0)
 			(effects
@@
 			)
 		)
-		(property "Footprint" "TBP01R250806BE"
+		(property "Footprint" "InverterCom:TBP01R250806BE"
 			(at 31.75 7.95 0)
 			(effects
@@
 			)
 		)
-		(property "Footprint" "MountingHole:MountingHole_5.3mm_M5"
+		(property "Footprint" "MountingHole:MountingHole_4.3mm_M4"
 			(at 254 67.31 0)
 			(effects
