File: Boards/ControlBoard/ControlBoard.kicad_pcb (KiCad board)
At the start: 6 copper layers, 297.5 x 60 mm, 140 parts, among them IC3 MAX22530AWE+, IC4 MAX22530AWE+, J1 TBP02R2W-381-06BE, J11 Conn_02x10_Counter_Clockwise, J12 Conn_02x10_Counter_Clockwise, J13 Conn_02x10_Counter_Clockwise, J14 Conn_02x10_Counter_Clockwise, J2 TBP02R2W-381-06BE, J23 776231-1, J29 Conn_01x02_Pin, J3 TBP01R2W-508-02BE, J4 TBP01R1-508-04BE, J5 Conn_02x10_Counter_Clockwise, J7 TBP02R2W-381-08BE, J8 TBP02R2W-381-08BE

Commit message: layout control boards, add baseplate, refine mechanical layout
Parts:
- removed C154, C155, C168, C169, C170, C171: UCM1H101MCL1GS, InverterCom:CAPAE660X800N
- removed C22, C24: 1uF, Capacitor_SMD:C_1210_3225Metric_Pad1.33x2.70mm_HandSolder
- removed J23: 776231-1, InverterCom:7762311
- removed LED11, LED12, LED36, LED37: LTST-C230GKT, InverterCom:LEDC3216X120N
- removed R126, R127, R23: 220, Resistor_SMD:R_1210_3225Metric_Pad1.30x2.65mm_HandSolder
- removed R24: 1k, Resistor_SMD:R_1210_3225Metric_Pad1.30x2.65mm_HandSolder
- removed TP13, TP14, TP15, TP16, TP17, TP18, TP19, TP20: TestPoint, TestPoint:TestPoint_Loop_D2.54mm_Drill1.5mm_Beaded
- added D4: S3N, InverterCom:DIOM8059X265N, B.Cu at (9.55, 37.0)
- added R13: 10k, Resistor_SMD:R_1210_3225Metric_Pad1.30x2.65mm_HandSolder, B.Cu at (177.9, 4.50)
- C132, C133, C14, C140, C141, C142, C143, C144, C145, C146, C147, C148, C149, C15, C150, C151, C152, C153, C16, C18, C20, C21, C23, C49, C50, C51, C52, F1, R12: moved to B.Cu
- moved LED3 234.4 mm to (175.5, 24.5)
- moved TP12 223.2 mm to (165.5, 14.0), turned to 90 degrees
- moved C167 220.5 mm to (106.3, 5.00), turned to 90 degrees
- moved C148 219.8 mm to (106.3, 5.00), turned to 90 degrees
- moved C149 214.4 mm to (98.5, 5.00), turned to 90 degrees
- moved C166 210.3 mm to (98.5, 5.00), turned to 90 degrees
- moved C150 209.5 mm to (90.7, 5.00), turned to 90 degrees
- moved R6 206.8 mm to (180.5, 24.5)
- moved C151 205.0 mm to (82.9, 5.00), turned to 90 degrees
- moved C165 200.2 mm to (90.7, 5.00), turned to 90 degrees
- moved TP11 198.2 mm to (141.0, 14.0), turned to 90 degrees
- moved C164 190.2 mm to (82.9, 5.00), turned to 90 degrees
- moved C20 189.1 mm to (161.0, 27.5), turned to 180 degrees
- moved C16 188.0 mm to (155.1, 34.0), turned to 180 degrees
- moved LED4 187.8 mm to (121.5, 10.5), turned to -90 degrees
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Connections:
- A1 pad 11: /Control/GATE_DRIVER_READY_A -> /READY
- A1 pad 12: /Control/GATE_DRIVER_RESET_A -> /RESET
- A1 pad 31: /Control/GATE_DRIVER_FAULT_A -> /FAULT
- J13 pad 7: unconnected-(J13-Pin_7-Pad7) -> /RESET
- J13 pad 8: unconnected-(J13-Pin_8-Pad8) -> /READY
- J13 pad 9: unconnected-(J13-Pin_9-Pad9) -> /FAULT
Other:
- outline, holes or cut-outs redrawn
- board text added: "important! replace pi pico footprint with one without antenna keepout, using the 2.54mm headers"

Commit message: Layout controlboard, update cad
Parts:
- removed TP25, TP26, TP27, TP28: TestPoint, TestPoint:TestPoint_Loop_D2.54mm_Drill1.5mm_Beaded
- added C154: UCM1H101MCL1GS, InverterCom:CAPAE660X800N, F.Cu at (247.3, 5.90)
- added C155: UCM1H101MCL1GS, InverterCom:CAPAE660X800N, F.Cu at (247.3, 13.7)
- added C156: UCM1H101MCL1GS, InverterCom:CAPAE660X800N, F.Cu at (247.3, 21.5)
- added C157: UCM1H101MCL1GS, InverterCom:CAPAE660X800N, F.Cu at (247.3, 29.3)
- added C158: UCM1H101MCL1GS, InverterCom:CAPAE660X800N, F.Cu at (239.4, 39.3)
- added C159: UCM1H101MCL1GS, InverterCom:CAPAE660X800N, F.Cu at (239.4, 47.1)
- added C160: UCM1H101MCL1GS, InverterCom:CAPAE660X800N, F.Cu at (239.4, 54.9)
- added C161: UCM1H101MCL1GS, InverterCom:CAPAE660X800N, F.Cu at (249.3, 39.3)
- added C162: UCM1H101MCL1GS, InverterCom:CAPAE660X800N, F.Cu at (249.3, 47.1)
- added C163: UCM1H101MCL1GS, InverterCom:CAPAE660X800N, F.Cu at (249.3, 54.9)
- added C168: UCM1H101MCL1GS, InverterCom:CAPAE660X800N, F.Cu at (257.2, 29.4)
- added C169: UCM1H101MCL1GS, InverterCom:CAPAE660X800N, F.Cu at (257.2, 5.90)
- added C170: UCM1H101MCL1GS, InverterCom:CAPAE660X800N, F.Cu at (257.2, 13.7)
- added C171: UCM1H101MCL1GS, InverterCom:CAPAE660X800N, F.Cu at (257.2, 21.5)
- added C172: UCM1H101MCL1GS, InverterCom:CAPAE660X800N, F.Cu at (259.2, 39.3)
- added C173: UCM1H101MCL1GS, InverterCom:CAPAE660X800N, F.Cu at (259.2, 47.1)
- added C174: UCM1H101MCL1GS, InverterCom:CAPAE660X800N, F.Cu at (259.2, 54.9)
- added C175: UCM1H101MCL1GS, InverterCom:CAPAE660X800N, F.Cu at (269.1, 39.3)
- added C176: UCM1H101MCL1GS, InverterCom:CAPAE660X800N, F.Cu at (269.1, 47.1)
- added C177: UCM1H101MCL1GS, InverterCom:CAPAE660X800N, F.Cu at (269.1, 54.9)
- added G***: LOGO, InverterCom:HIGHVOLTAGE_20mm, F.Cu at (115.0, 47.0)
- A1: footprint InverterCom:RaspberryPi_Pico_Common_Unspecified -> Module:RaspberryPi_Pico_Common_THT
- C120, C123: moved to F.Cu
- C121, C13, Z13, Z16: moved to B.Cu
- moved TP29 73.1 mm to (193.0, 56.5)
- moved TP32 61.6 mm to (186.5, 56.5)
- moved TP24 54.0 mm to (61.0, 49.5)
- moved TP31 52.0 mm to (176.5, 56.5)
- moved TP35 51.5 mm to (181.5, 56.5)
- moved TP22 43.3 mm to (66.5, 49.5)
- moved TP30 43.1 mm to (166.5, 56.5)
- moved TP34 42.0 mm to (171.5, 56.5)
- moved TP21 37.6 mm to (72.5, 49.5)
- moved TP33 33.6 mm to (161.5, 56.5)
- moved TP23 31.8 mm to (78.5, 49.5)
- moved A1 25.9 mm to (104.8, 16.6)
- moved Z14 8.83 mm to (138.0, 14.3), turned to -90 degrees
- moved C121 6.75 mm to (135.9, 19.0)
- moved C122 6.19 mm to (129.0, 15.9), turned to -90 degrees
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Connections:
- A1 pad 21: /SPI2_ADC4_CS_A -> /PH_U_L
- A1 pad 22: /PH_U_L -> /PH_U_H
- A1 pad 25: /PH_W_L -> /PH_V_H
- A1 pad 26: /PH_U_H -> /PH_W_L
- A1 pad 27: /PH_V_H -> /PH_W_H
- A1 pad 29: /PH_W_H -> /SPI2_ADC4_CS_A
- J1 pad 2: /SPARE_V -> /THROTTLE_V
- J1 pad 3: /REGEN_THROTTLE_V -> /SPARE_V
- J1 pad 4: /THROTTLE_V -> /REGEN_THROTTLE_V
- J14 pad 5: /CAN_5V_OUT -> unconnected-(J14-Pin_5-Pad5)
- J5 pad 16: /+12V_A -> unconnected-(J5-Pin_16-Pad16)
- J5 pad 19: /+12V_SWITCHED_A -> unconnected-(J5-Pin_19-Pad19)
- J7 pad 5: /CAN_5V_OUT -> unconnected-(J7-Pad5)
- J8 pad 1: /+12V_SWITCHED_A -> unconnected-(J8-Pad1)
- J8 pad 2: /+12V_A -> unconnected-(J8-Pad2)
Routing:
- net /RELAY_2_A: track 0.00 -> 249.4 mm, vias 0 -> 5
- net /RELAY_3_A: track 0.00 -> 248.7 mm, vias 0 -> 5
- net /RELAY_1_A: track 0.00 -> 238.8 mm, vias 0 -> 4
- net /PH_W_L: track 0.00 -> 153.7 mm, vias 0 -> 5
- net /PH_W_H: track 0.00 -> 152.5 mm, vias 0 -> 5
- net /PH_V_H: track 0.00 -> 141.9 mm, vias 0 -> 5
- net /SPI2_RX_A: track 0.00 -> 140.1 mm, vias 0 -> 6
- net /PH_V_L: track 0.00 -> 139.0 mm, vias 0 -> 5
- net /PH_U_L: track 0.00 -> 134.9 mm, vias 0 -> 5
- net /PH_U_H: track 0.00 -> 131.5 mm, vias 0 -> 5
- net /SPI2_SCK_A: track 0.00 -> 130.6 mm, vias 0 -> 4
- net /SPI2_TX_A: track 0.00 -> 129.6 mm, vias 0 -> 5
- net /RESET: track 0.00 -> 125.3 mm, vias 0 -> 4
- net /READY: track 0.00 -> 119.5 mm, vias 0 -> 4
- net /SPI2_ADC3_CS_A: track 0.00 -> 103.2 mm, vias 0 -> 5
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- added copper zone on In3.Cu, net /+12V_A
- added copper zone on In2.Cu, net /+3.3V_A
- added copper zone on In2.Cu, net /+5V_V
- added copper zone on In2.Cu, net /+5V_W
- added copper zone on B.Cu, net /CAN_GND
- added copper zone on F.Cu, net /CAN_GND
- added copper zone on In1.Cu, net /CAN_GND
- added copper zone on In4.Cu, net /CAN_GND
- added copper zone on B.Cu, net /GND_A
- added copper zone on F.Cu, net /GND_A
- added copper zone on In1.Cu, net /GND_A
- added copper zone on In4.Cu, net /GND_A
- added copper zone on B.Cu, net /GND_V
- added copper zone on F.Cu, net /GND_V
- added copper zone on In1.Cu, net /GND_V
- added copper zone on In4.Cu, net /GND_V
- added copper zone on B.Cu, net /GND_W
- added copper zone on F.Cu, net /GND_W
- added copper zone on In1.Cu, net /GND_W
- added copper zone on In4.Cu, net /GND_W
- added copper zone on B.Cu, net /Power/GND_Z
- added copper zone on F.Cu, net /Power/GND_Z
- added copper zone on In1.Cu, net /Power/GND_Z
- added copper zone on In4.Cu, net /Power/GND_Z
- added copper zone on In2.Cu, net Net-(C140-+)
- added copper zone on In3.Cu, net Net-(C140-+)
Other:
- board text added: "DANGER! HAZARDOUS VOLTAGES PRESENT REMOVE POWER AND VERIFY CAPACITORS DISCHARGED BEFORE SERVICING"
- board text added: "DESIGNED BY THOMAS LIAO"
- board text added: "ISOLATION BARRIER DO NOT CROSS"
- board text added: "TRACTION INVERTER, GEN 5, CONTROL BOARD, REVISION 1, 1200VMAX, 800V WORKING"
- board text removed: "important! replace pi pico footprint with one without antenna keepout, using the 2.54mm headers"

Commit message: fix connector pinout
Other:
- board text added: "+5V H_U H_W H_V MTRTMP GND"
- board text added: "+5V NC RGN SPRE THRT GND"
- board text added: "1->"
- board text added: "<-1"
- board text added: "GND CH CL NC +24v NC CJPA CJPB"
- board text added: "GND VIN (9-18V)"
- board text added: "NC GND HS_TMP +5V"
- board text added: "R1NO R1COM R2COM R2NO R3COM R3NO NC NC"
Changed lines of the file:
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@@
 		(tags "Connector")
 		(property "Reference" "J8"
-			(at 13.335 -5.5 90)
+			(at -8.57 0 90)
 			(layer "F.SilkS")
 			(effects
@@
 			(fill no)
 			(layer "Cmts.User")
-			(net 47)
 		)
 		(fp_circle
@@
 			(fill no)
 			(layer "F.CrtYd")
-			(net 47)
 		)
 		(fp_text user "${REFERENCE}"
@@
 			(fill no)
 			(layer "Cmts.User")
-			(net 47)
 		)
 		(fp_circle
@@
 			(fill no)
 			(layer "F.CrtYd")
-			(net 47)
 		)
 		(fp_text user "${REFERENCE}"
@@
 			(fill no)
 			(layer "Cmts.User")
-			(net 47)
 		)
 		(fp_circle
@@
 			(fill no)
 			(layer "F.CrtYd")
-			(net 47)
 		)
 		(fp_text user "${REFERENCE}"
@@
 			(fill no)
 			(layer "Cmts.User")
-			(net 47)
 		)
 		(fp_circle
@@
 			(fill no)
 			(layer "F.CrtYd")
-			(net 47)
 		)
 		(fp_text user "${REFERENCE}"
@@
 			(fill no)
 			(layer "Cmts.User")
-			(net 47)
 		)
 		(fp_circle
@@
 			(fill no)
 			(layer "F.CrtYd")
-			(net 47)
 		)
 		(fp_text user "${REFERENCE}"
@@
 			(fill no)
 			(layer "Cmts.User")
-			(net 47)
 		)
 		(fp_circle
@@
 			(fill no)
 			(layer "F.CrtYd")
-			(net 47)
 		)
 		(fp_text user "${REFERENCE}"
@@
 		(tags "Connector")
 		(property "Reference" "J4"
-			(at 7.5 -3.5 180)
+			(at -4.88 7 180)
 			(layer "B.SilkS")
 			(effects
@@
 		)
 	)
+	(gr_text "1->"
+		(at 195 0 270)
+		(layer "F.SilkS")
+		(effects
+			(font
+				(size 1 1)
+				(thickness 0.25)
+				(bold yes)
+			)
+			(justify left bottom)
+		)
+	)
 	(gr_text "DANGER!\nHAZARDOUS VOLTAGES PRESENT\nREMOVE POWER AND VERIFY\nCAPACITORS DISCHARGED BEFORE SERVICING"
 		(at 124 54 0)
@@
 		)
 	)
+	(gr_text "1->"
+		(at 230.5 5.5 0)
+		(layer "F.SilkS")
+		(effects
+			(font
+				(size 1 1)
+				(thickness 0.25)
+				(bold yes)
+			)
+			(justify left bottom)
+		)
+	)
 	(gr_text "ISOLATION BARRIER DO NOT CROSS"
 		(at 191 30 90)
@@
 		)
 	)
+	(gr_text "GND   VIN\n(9-18V)"
+		(at 1 23 270)
+		(layer "F.SilkS")
+		(effects
+			(font
+				(size 1.5 1)
+				(thickness 0.25)
+				(bold yes)
+			)
+			(justify bottom)
+		)
+	)
+	(gr_text "<-1"
+		(at 85 40.5 0)
+		(layer "F.SilkS")
+		(effects
+			(font
+				(size 1 1)
+				(thickness 0.25)
+				(bold yes)
+			)
+			(justify left bottom)
+		)
+	)
 	(gr_text "TRACTION INVERTER, GEN 5,\nCONTROL BOARD,\nREVISION 1,\n1200VMAX, 800V WORKING"
 		(at 197 58 0)
@@
 		)
 	)
+	(gr_text "GND  CH  CL  NC  +24v NC CJPA CJPB"
+		(at 211 39 90)
+		(layer "F.SilkS")
+		(effects
+			(font
+				(size 1.5 1)
+				(thickness 0.25)
+				(bold yes)
+			)
+			(justify left bottom)
+		)
+	)
+	(gr_text "<-1"
+		(at 160 42 0)
+		(layer "F.SilkS")
+		(effects
+			(font
+				(size 1 1)
+				(thickness 0.25)
+				(bold yes)
+			)
+			(justify left bottom)
+		)
+	)
+	(gr_text "R1NO R1COM R2COM R2NO R3COM R3NO   NC   NC"
+		(at 286 48 90)
+		(layer "F.SilkS")
+		(effects
+			(font
+				(size 1.5 0.75)
+				(thickness 0.1875)
+				(bold yes)
+			)
+			(justify left bottom)
+		)
+	)
+	(gr_text "1->"
+		(at 286.5 17.5 0)
+		(layer "F.SilkS")
+		(effects
+			(font
+				(size 1 1)
+				(thickness 0.25)
+				(bold yes)
+			)
+			(justify left bottom)
+		)
+	)
+	(gr_text "+5V H_U H_W H_V MTRTMP GND"
+		(at 141 3 0)
+		(layer "B.SilkS")
+		(effects
+			(font
+				(size 1.5 1)
+				(thickness 0.25)
+				(bold yes)
+			)
+			(justify left bottom mirror)
+		)
+	)
+	(gr_text "+5V NC RGN SPRE THRT GND"
+		(at 175 3 0)
+		(layer "B.SilkS")
+		(effects
+			(font
+				(size 1.5 1)
+				(thickness 0.25)
+				(bold yes)
+			)
+			(justify left bottom mirror)
+		)
+	)
+	(gr_text "NC GND HS_TMP +5V"
+		(at 187 8 0)
+		(layer "B.SilkS")
+		(effects
+			(font
+				(size 1.5 1)
+				(thickness 0.25)
+				(bold yes)
+			)
+			(justify left bottom mirror)
+		)
+	)
