File: Boards/ControlBoard/ControlBoard.kicad_pcb (KiCad board)
At the start: 6 copper layers, 297.5 x 60 mm, 134 parts, among them IC3 MAX22530AWE+, IC4 MAX22530AWE+, J1 TBP02R2W-381-06BE, J11 Conn_02x10_Counter_Clockwise, J12 Conn_02x10_Counter_Clockwise, J13 Conn_02x10_Counter_Clockwise, J14 Conn_02x10_Counter_Clockwise, J2 TBP02R2W-381-06BE, J29 Conn_01x02_Pin, J3 TBP01R2W-508-02BE, J4 TBP01R1-508-04BE, J5 Conn_02x10_Counter_Clockwise, J7 TBP02R2W-381-08BE, J8 TBP02R2W-381-08BE

Commit message: Add Clearance To Main/CtrlBd, Increase main DCDC to 20w
Parts:
- removed PS7: NSD15-12S12, InverterCom:NSD1512S12
- added C178: UCM1H101MCL1GS, InverterCom:CAPAE660X800N, F.Cu at (40.4, 45.0)
- added C179: UCM1H101MCL1GS, InverterCom:CAPAE660X800N, F.Cu at (40.4, 54.0)
- added C180: UCM1H101MCL1GS, InverterCom:CAPAE660X800N, B.Cu at (40.4, 54.0)
- added C181: UCM1H101MCL1GS, InverterCom:CAPAE660X800N, F.Cu at (30.4, 43.5)
- added PS1: SCW20A-12, InverterCom:SCW20A12, F.Cu at (33.7, 37.3)
- C145, C147: moved to F.Cu
- H1, H7: footprint MountingHole:MountingHole_5.3mm_M5 -> MountingHole:MountingHole_3.2mm_M3
- H3, H4, H5, H8: footprint MountingHole:MountingHole_5.3mm_M5 -> MountingHole:MountingHole_4.3mm_M4
- moved C173 41.8 mm to (267.0, 6.00)
- moved C174 41.8 mm to (267.0, 13.8)
- moved C50 29.4 mm to (17.0, 29.5)
- moved C176 26.0 mm to (267.0, 21.2)
- moved C177 26.0 mm to (267.0, 29.0)
- moved C49 24.9 mm to (21.5, 35.4), turned to 90 degrees
- moved H7 24.7 mm to (266.5, 51.0)
- moved C147 21.3 mm to (44.9, 10.0)
- moved C145 20.6 mm to (44.1, 19.5)
- moved H1 16.3 mm to (23.5, 51.0)
- moved C153 10.3 mm to (26.0, 6.50), turned to 90 degrees
- moved C146 9.31 mm to (26.0, 17.0), turned to 90 degrees
- moved J8 8.63 mm to (279.0, 10.0)
- moved C141 7.76 mm to (27.9, 34.0), turned to 0 degrees
- moved C142 2.92 mm to (18.9, 42.5)
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Connections:
- net Net-(C140-+) renamed /Power/VIN_FUSED_Z
Routing:
- net /RELAY3_COM: track 41.7 -> 33.6 mm
- net /RELAY3_NO: track 20.2 -> 12.3 mm, vias 2 -> 0
- net /RELAY2_NO: track 22.6 -> 14.8 mm, vias 1 -> 2
- net /RELAY1_NO: track 28.2 -> 20.7 mm, vias 2 -> 1
- net /RELAY1_COM: track 31.6 -> 38.6 mm
- net /RELAY2_COM: track 42.4 -> 49.1 mm, vias 4 -> 2
- net /Power/VIN_FUSED_Z: track 15.5 -> 20.4 mm, vias 8 -> 9
- net /Power/GND_Z: vias 0 -> 1
- net /+12V_A: vias 20 -> 18
Other:
- outline, holes or cut-outs redrawn
- board text added: "GND VIN (10-16V)"
- board text added: "ISOLATION BARRIER"
- board text removed: "GND VIN (9-18V)"
