File: Boards/ControlBoard/ControlBoard.kicad_sch (KiCad schematic)
At the start: 12 parts, among them J1 TBP02R2W-381-06BE, J11 Conn_02x10_Counter_Clockwise, J12 Conn_02x10_Counter_Clockwise, J13 Conn_02x10_Counter_Clockwise, J14 Conn_02x10_Counter_Clockwise, J2 TBP02R2W-381-06BE, J3 TBP01R2W-508-02BE, J4 TBP01R1-508-04BE, J5 Conn_02x10_Counter_Clockwise, J7 TBP02R2W-381-08BE, J8 TBP02R2W-381-08BE

Commit message: Add Clearance To Main/CtrlBd, Increase main DCDC to 20w
Parts:
- added H1, H7: MountingHole, MountingHole:MountingHole_3.2mm_M3, symbol Mechanical:MountingHole
- added H3, H4, H5, H8: MountingHole, MountingHole:MountingHole_4.3mm_M4, symbol Mechanical:MountingHole
- J1, J2: footprint TBP02R2W38106BE -> InverterCom:TBP02R2W38106BE
- J3: footprint TBP01R2W50802BE -> InverterCom:TBP01R2W50802BE
- J4: footprint TBP01R150804BE -> InverterCom:TBP01R150804BE
