File: Boards/ControlBoard/Power.kicad_sch (KiCad schematic)
At the start: 47 parts

Commit message: Add Clearance To Main/CtrlBd, Increase main DCDC to 20w
Parts:
- removed PS7: NSD15-12S12, InverterCom:NSD1512S12, symbol InverterCom:NSD15-12S12
- added C178, C179, C180, C181: UCM1H101MCL1GS, InverterCom:CAPAE660X800N, symbol InverterCom:UCM1H101MCL1GS
- added PS1: SCW20A-12, InverterCom:SCW20A12, symbol InverterCom:SCW20A-12
Connections:
- net +12V_OUT_A: now also PS1.14 (+VOUT)
- net GND_A: now also PS1.16 (-VOUT)
- net GND_Z: now also C178.2 (-), C179.2 (-), C180.2 (-), C181.2 (-), PS1.2 (-VIN_1), PS1.3 (-VIN_2)
- net VIN_FUSED_Z: now reaches C140.1 (+), C141.1 (+), C142.1 (+), C143.1 (+), C49.2, C50.2, D3.1 (K), D4.1 (K)
- net VIN_FUSED_Z: now also C178.1 (+), C179.1 (+), C180.1 (+), C181.1 (+), PS1.22 (+VIN_1), PS1.23 (+VIN_2)
- no-connect marks 3 -> 4
Other:
- note added: "VIN IS 9-18V ONLY"
- note removed: "VIN IS 9-36V ONLY"
- moved on the sheet: C140, C141, C142, C143, C49, C50, C51, C52, D3, D4, F1, PS6
